File: steny_pcb/steny.kicad_sch (KiCad schematic)
At the start: 0 parts

Commit message: progress can be seen in the JOURNAL.md file.
Parts:
- added A1: RaspberryPi_Pico, Module:RaspberryPi_Pico_Common_Unspecified, symbol MCU_Module:RaspberryPi_Pico
- added CP1, CP10, CP11, CP12, CP13, CP14, CP15, CP16, CP17, CP18, CP19, CP2, CP20, CP21, CP22, CP3, CP4, CP5, CP6, CP7, CP8, CP9: Copper Pad 14.5x16.5, customs:copper_pad_14_5x16_5, symbol custom:copper_pad_14_5x16_5
- added CP23, CP24, CP25: Copper Pad 14.5x33, customs:copper_pad_14_5x33, symbol custom:copper_pad_14_5x33
Connections:
- new net: A1.9 (GPIO6), CP14.1 (TP)
- new net: A1.26 (GPIO20), CP11.1 (TP)
- new net: A1.4 (GPIO2), CP12.1 (TP)
- new net: A1.12 (GPIO9), CP5.1 (TP)
- new net: A1.19 (GPIO14), CP18.1 (TP)
- new net: A1.10 (GPIO7), CP4.1 (TP)
- new net: A1.22 (GPIO17), CP20.1 (TP)
- new net: A1.24 (GPIO18), CP10.1 (TP)
- new net: A1.25 (GPIO19), CP21.1 (TP)
- new net: A1.16 (GPIO12), CP17.1 (TP)
- new net: A1.2 (GPIO1), CP1.1 (TP)
- new net: A1.1 (GPIO0), CP25.1 (TP)
- new net: A1.21 (GPIO16), CP9.1 (TP)
- new net: A1.15 (GPIO11), CP6.1 (TP)
- new net: A1.11 (GPIO8), CP15.1 (TP)
- new net: A1.13 (GND), A1.18 (GND), A1.23 (GND), A1.28 (GND), A1.3 (GND), A1.38 (GND), A1.8 (GND)
- new net: A1.14 (GPIO10), CP16.1 (TP)
- new net: A1.17 (GPIO13), CP7.1 (TP)
- new net: A1.20 (GPIO15), CP8.1 (TP)
- new net: A1.27 (GPIO21), CP22.1 (TP)
- new net: A1.31 (GPIO26_ADC0), CP23.1 (TP)
- new net: A1.32 (GPIO27_ADC1), CP24.1 (TP)
- new net: A1.5 (GPIO3), CP2.1 (TP)
- new net: A1.6 (GPIO4), CP13.1 (TP)
- new net: A1.7 (GPIO5), CP3.1 (TP)

Commit message: Finished PCB
Parts:
- CP23, CP24, CP25: value Copper Pad 14.5x33 -> Copper Pad 14.5x38; footprint customs:copper_pad_14_5x33 -> customs:copper_pad_14_5x38
Connections:
- net at CP19.1 (TP): now also A1.29 (GPIO22)
- no-connect marks 0 -> 6
Changed lines of the file:
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@@
 	(generator_version "9.0")
 	(paper "A4")
+	(no_connect
+		(at 1.27 274.32)
+	)
+	(no_connect
+		(at 24.13 53.34)
+	)
+	(no_connect
+		(at 49.53 245.11)
+	)
+	(no_connect
+		(at 50.8 109.22)
+	)
+	(no_connect
+		(at 44.45 57.15)
+	)
+	(no_connect
+		(at 2.54 168.91)
+	)
 	(wire
 		(pts
@@
 	(wire
 		(pts
+			(xy 262.89 115.57) (xy 262.89 81.28)
+		)
+		(stroke
+			(width 0)
+			(type default)
+		)
+	)
+	(wire
+		(pts
 			(xy 129.54 85.09) (xy 186.69 85.09)
 		)
@@
 	(wire
 		(pts
+			(xy 262.89 81.28) (xy 245.11 81.28)
+		)
+		(stroke
+			(width 0)
+			(type default)
+		)
+	)
+	(wire
+		(pts
 			(xy 129.54 123.19) (xy 250.19 123.19)
 		)
@@
 		(pts
 			(xy 109.22 134.62) (xy 257.81 134.62)
+		)
+		(stroke
+			(width 0)
+			(type default)
+		)
+	)
+	(wire
+		(pts
+			(xy 129.54 115.57) (xy 262.89 115.57)
 		)
 		(stroke
@@
 		(on_board yes)
 		(dnp no)
-		(fields_autoplaced yes)
 		(property "Reference" "CP25"
-			(at 190.5 22.8601 90)
-			(effects
-				(font
-					(size 1.27 1.27)
-				)
-				(justify right)
-			)
-		)
-		(property "Value" "Copper Pad 14.5x33"
-			(at 190.5 20.3201 90)
-			(effects
-				(font
-					(size 1.27 1.27)
-				)
-				(justify right)
-			)
-		)
-		(property "Footprint" "customs:copper_pad_14_5x33"
+			(at 185.674 22.606 90)
+			(effects
+				(font
+					(size 1.27 1.27)
+				)
+				(justify left)
+			)
+		)
+		(property "Value" "Copper Pad 14.5x38"
+			(at 170.688 19.812 90)
+			(effects
+				(font
+					(size 1.27 1.27)
+				)
+				(justify left)
+			)
+		)
+		(property "Footprint" "customs:copper_pad_14_5x38"
 			(at 190.5 21.59 0)
 			(effects
@@
 		(on_board yes)
 		(dnp no)
-		(fields_autoplaced yes)
 		(property "Reference" "CP24"
 			(at 218.44 22.8601 90)
@@
 			)
 		)
-		(property "Value" "Copper Pad 14.5x33"
+		(property "Value" "Copper Pad 14.5x38"
 			(at 218.44 20.3201 90)
 			(effects
@@
 			)
 		)
-		(property "Footprint" "customs:copper_pad_14_5x33"
+		(property "Footprint" "customs:copper_pad_14_5x38"
 			(at 218.44 21.59 0)
 			(effects
@@
 		(on_board yes)
 		(dnp no)
-		(fields_autoplaced yes)
 		(property "Reference" "CP23"
-			(at 246.38 22.8601 90)
-			(effects
-				(font
-					(size 1.27 1.27)
-				)
-				(justify right)
-			)
-		)
-		(property "Value" "Copper Pad 14.5x33"
-			(at 246.38 20.3201 90)
-			(effects
-				(font
-					(size 1.27 1.27)
-				)
-				(justify right)
-			)
-		)
-		(property "Footprint" "customs:copper_pad_14_5x33"
+			(at 241.554 22.86 90)
+			(effects
+				(font
+					(size 1.27 1.27)
+				)
+				(justify left)
+			)
+		)
+		(property "Value" "Copper Pad 14.5x38"
+			(at 226.822 20.32 90)
+			(effects
+				(font
+					(size 1.27 1.27)
+				)
+				(justify left)
+			)
+		)
+		(property "Footprint" "customs:copper_pad_14_5x38"
 			(at 246.38 21.59 0)
 			(effects
